Commit message: Migrate Mark's autonomy stack: lane detection, LiDAR obstacles, NML waypoints, joy bridge

File: ros2_ws_mark/src/littleblue_sim/urdf/gazebo_plugins.xacro (robot description, xacro)
@@ -11,5 +11,5 @@
       <max_linear_acceleration>1.0</max_linear_acceleration>
       <max_angular_acceleration>2.0</max_angular_acceleration>
-      <odom_publish_frequency>30</odom_publish_frequency>
+      <odom_publish_frequency>100</odom_publish_frequency>
       <topic>cmd_vel</topic>
       <odom_topic>odom</odom_topic>
@@ -31,12 +31,12 @@
     <mu2>0.0</mu2>
   </gazebo>
-  <!-- RGB Camera sensor -->
-  <gazebo reference="camera_link">
-    <sensor name="rgb_camera" type="camera">
+  <!-- Left RGB Camera sensor -->
+  <gazebo reference="left_camera_link">
+    <sensor name="left_rgb_camera" type="camera">
       <always_on>true</always_on>
       <update_rate>15</update_rate>
-      <topic>image_raw</topic>
+      <topic>left_camera/image_raw</topic>
       <camera>
-        <horizontal_fov>1.2112</horizontal_fov>
+        <horizontal_fov>1.4835</horizontal_fov>
         <image>
           <width>640</width>
@@ -51,20 +51,20 @@
     </sensor>
   </gazebo>
-  <!-- Depth Camera sensor -->
-  <gazebo reference="depth_camera_link">
-    <sensor name="depth_camera" type="depth_camera">
+  <!-- Right RGB Camera sensor -->
+  <gazebo reference="right_camera_link">
+    <sensor name="right_rgb_camera" type="camera">
       <always_on>true</always_on>
       <update_rate>15</update_rate>
-      <topic>depth/image_raw</topic>
+      <topic>right_camera/image_raw</topic>
       <camera>
-        <horizontal_fov>1.5184</horizontal_fov>
+        <horizontal_fov>1.4835</horizontal_fov>
         <image>
           <width>640</width>
           <height>480</height>
-          <format>R_FLOAT32</format>
+          <format>R8G8B8</format>
         </image>
         <clip>
           <near>0.1</near>
-          <far>10</far>
+          <far>100</far>
         </clip>
       </camera>
@@ -80,8 +80,8 @@
         <scan>
           <horizontal>
-            <samples>360</samples>
+            <samples>270</samples>
             <resolution>1</resolution>
-            <min_angle>-3.14159</min_angle>
-            <max_angle>3.14159</max_angle>
+            <min_angle>-2.35619</min_angle>
+            <max_angle>2.35619</max_angle>
           </horizontal>
           <vertical>
@@ -134,8 +134,8 @@
         <position_sensing>
           <horizontal>
-            <noise type="gaussian"><mean>0</mean><stddev>0.5</stddev></noise>
+            <noise type="gaussian"><mean>0</mean><stddev>0.000005</stddev></noise>
           </horizontal>
           <vertical>
-            <noise type="gaussian"><mean>0</mean><stddev>1.0</stddev></noise>
+            <noise type="gaussian"><mean>0</mean><stddev>0.00001</stddev></noise>
           </vertical>
         </position_sensing>

File: ros2_ws_mark/src/littleblue_sim/urdf/sensors.xacro (robot description, xacro)
@@ -1,51 +1,59 @@
 <?xml version="1.0"?>
 <robot xmlns:xacro="http://www.ros.org/wiki/xacro">
-  <!-- RGB Camera (front-facing, matching D435i FOV) -->
-  <link name="camera_link">
-    <visual>
-      <geometry>
-        <box size="0.03 0.09 0.025"/>
-      </geometry>
-      <material name="dark_grey"/>
-    </visual>
-    <collision>
-      <geometry>
-        <box size="0.03 0.09 0.025"/>
-      </geometry>
-    </collision>
-    <inertial>
-      <mass value="0.1"/>
-      <inertia ixx="0.0001" ixy="0" ixz="0" iyy="0.0001" iyz="0" izz="0.0001"/>
-    </inertial>
-  </link>
-  <joint name="camera_joint" type="fixed">
-    <parent link="base_link"/>
-    <child link="camera_link"/>
-    <origin xyz="${chassis_length/2 - 0.02} 0 ${chassis_height + 0.02}" rpy="0 0 0"/>
-  </joint>
-  <link name="camera_optical_link"/>
-  <joint name="camera_optical_joint" type="fixed">
-    <parent link="camera_link"/>
-    <child link="camera_optical_link"/>
-    <origin xyz="0 0 0" rpy="${-pi/2} 0 ${-pi/2}"/>
-  </joint>
-  <!-- Depth Camera (co-located with RGB) -->
-  <link name="depth_camera_link">
-    <inertial>
-      <mass value="0.01"/>
-      <inertia ixx="0.00001" ixy="0" ixz="0" iyy="0.00001" iyz="0" izz="0.00001"/>
-    </inertial>
-  </link>
-  <joint name="depth_camera_joint" type="fixed">
-    <parent link="camera_link"/>
-    <child link="depth_camera_link"/>
-    <origin xyz="0 0 0" rpy="0 0 0"/>
-  </joint>
-  <link name="depth_camera_optical_link"/>
-  <joint name="depth_camera_optical_joint" type="fixed">
-    <parent link="depth_camera_link"/>
-    <child link="depth_camera_optical_link"/>
-    <origin xyz="0 0 0" rpy="${-pi/2} 0 ${-pi/2}"/>
-  </joint>
+  <!-- Camera pair macro: creates RGB + depth links at a lateral offset -->
+  <xacro:macro name="camera_pair" params="prefix y_offset">
+    <!-- RGB Camera -->
+    <link name="${prefix}_camera_link">
+      <visual>
+        <geometry>
+          <box size="0.03 0.09 0.025"/>
+        </geometry>
+        <material name="dark_grey"/>
+      </visual>
+      <collision>
+        <geometry>
+          <box size="0.03 0.09 0.025"/>
+        </geometry>
+      </collision>
+      <inertial>
+        <mass value="0.1"/>
+        <inertia ixx="0.0001" ixy="0" ixz="0" iyy="0.0001" iyz="0" izz="0.0001"/>
+      </inertial>
+    </link>
+    <joint name="${prefix}_camera_joint" type="fixed">
+      <parent link="base_link"/>
+      <child link="${prefix}_camera_link"/>
+      <!-- Tilted down 5° (pitch=0.09) and outward 15° (yaw=±0.26) toward lane lines -->
+      <origin xyz="${chassis_length/2 - 0.02} ${y_offset} ${chassis_height + 0.02}" rpy="0 0.09 ${0.26 * y_offset/0.28}"/>
+    </joint>
+    <link name="${prefix}_camera_optical_link"/>
+    <joint name="${prefix}_camera_optical_joint" type="fixed">
+      <parent link="${prefix}_camera_link"/>
+      <child link="${prefix}_camera_optical_link"/>
+      <origin xyz="0 0 0" rpy="${-pi/2} 0 ${-pi/2}"/>
+    </joint>
+    <!-- Depth Camera (co-located with RGB) -->
+    <link name="${prefix}_depth_camera_link">
+      <inertial>
+        <mass value="0.01"/>
+        <inertia ixx="0.00001" ixy="0" ixz="0" iyy="0.00001" iyz="0" izz="0.00001"/>
+      </inertial>
+    </link>
+    <joint name="${prefix}_depth_camera_joint" type="fixed">
+      <parent link="${prefix}_camera_link"/>
+      <child link="${prefix}_depth_camera_link"/>
+      <origin xyz="0 0 0" rpy="0 0 0"/>
+    </joint>
+    <link name="${prefix}_depth_camera_optical_link"/>
+    <joint name="${prefix}_depth_camera_optical_joint" type="fixed">
+      <parent link="${prefix}_depth_camera_link"/>
+      <child link="${prefix}_depth_camera_optical_link"/>
+      <origin xyz="0 0 0" rpy="${-pi/2} 0 ${-pi/2}"/>
+    </joint>
+  </xacro:macro>
+  <!-- Left camera (+Y = left, chassis_width/2 - 0.02) -->
+  <xacro:camera_pair prefix="left" y_offset="0.28"/>
+  <!-- Right camera (-Y = right) -->
+  <xacro:camera_pair prefix="right" y_offset="-0.28"/>
   <!-- 2D LiDAR (top of chassis) -->
   <link name="lidar_link">
@@ -70,4 +78,27 @@
     <child link="lidar_link"/>
     <origin xyz="0 0 ${chassis_height + 0.05}" rpy="0 0 0"/>
+  </joint>
+  <!-- Rear electronics box — blocks ~90° of LiDAR behind the robot -->
+  <link name="rear_electronics_link">
+    <visual>
+      <geometry>
+        <box size="0.15 0.25 0.12"/>
+      </geometry>
+      <material name="dark_grey"/>
+    </visual>
+    <collision>
+      <geometry>
+        <box size="0.15 0.25 0.12"/>
+      </geometry>
+    </collision>
+    <inertial>
+      <mass value="0.5"/>
+      <inertia ixx="0.001" ixy="0" ixz="0" iyy="0.001" iyz="0" izz="0.001"/>
+    </inertial>
+  </link>
+  <joint name="rear_electronics_joint" type="fixed">
+    <parent link="base_link"/>
+    <child link="rear_electronics_link"/>
+    <origin xyz="${-chassis_length/4} 0 ${chassis_height + 0.06}" rpy="0 0 0"/>
   </joint>
   <!-- IMU (chassis center) -->
